Commit message: Condigured some code to my uses and joystick works now.
Signed-off-by: lidorshimoni <lidor.shim@gmail.com>

File: urdf/ABot.urdf.xacro (robot description, xacro)
@@ -140,5 +140,5 @@
     <origin rpy="1.5707963267948966 0 0" xyz="0 0 0"/>
     <geometry>
-      <sphere length="0.1" radius="0.025"/>
+      <sphere length="0.1" radius="0.05"/>
     </geometry>
   </visual>

Commit message: Added Move_Base control and keyboard control.
Signed-off-by: lidorshimoni <lidor.shim@gmail.com>

File: urdf/ABot.urdf.xacro (robot description, xacro)
@@ -140,11 +140,11 @@
     <origin rpy="1.5707963267948966 0 0" xyz="0 0 0"/>
     <geometry>
-      <sphere length="0.1" radius="0.05"/>
-    </geometry>
-  </visual>
-  <collision>
-    <origin rpy="1.5707963267948966 0 0" xyz="0 0 0"/>
-    <geometry>
-      <sphere length="0.1" radius="0.025"/>
+      <sphere length="0.1" radius="0.03"/>
+    </geometry>
+  </visual>
+  <collision>
+    <origin rpy="1.5707963267948966 0 0" xyz="0 0 0"/>
+    <geometry>
+      <sphere length="0.1" radius="0.03"/>
     </geometry>
   </collision>

Commit message: deleted move_base_test and now move_base gets a goal
Signed-off-by: lidorshimoni <lidor.shim@gmail.com>

File: urdf/ABot.urdf.xacro (robot description, xacro)
@@ -9,40 +9,40 @@
    </joint>-->
   <link name="base_link">
-  <inertial>
-    <origin xyz="0 0 0.125" />
-    <mass value="5" />
-    <inertia  ixx="0.1" ixy="0.0"  ixz="0.0"  iyy="0.1"  iyz="0.0"  izz="0.1" />
-  </inertial>
-  <visual>
-    <origin xyz="0 0 0.125"/>
-    <geometry>
-      <box size="0.4 0.2 0.1" />
-    </geometry>
-  </visual>
-  <collision>
-    <origin xyz="0 0 0.125"/>
-    <geometry>
-      <box size="0.4 0.2 0.1" />
-    </geometry>
-  </collision>
+    <inertial>
+      <origin xyz="0 0 0.125" />
+      <mass value="5" />
+      <inertia  ixx="0.1" ixy="0.0"  ixz="0.0"  iyy="0.1"  iyz="0.0"  izz="0.1" />
+    </inertial>
+    <visual>
+      <origin xyz="0 0 0.125"/>
+      <geometry>
+        <box size="0.4 0.2 0.1" />
+      </geometry>
+    </visual>
+    <collision>
+      <origin xyz="0 0 0.125"/>
+      <geometry>
+        <box size="0.4 0.2 0.1" />
+      </geometry>
+    </collision>
   </link>
   <link name="box">
-  <inertial>
-    <origin xyz="0 0 0" />
-    <mass value="5" />
-    <inertia  ixx="0.1" ixy="0.0"  ixz="0.0"  iyy="0.1"  iyz="0.0"  izz="0.1" />
-  </inertial>
-  <visual>
-    <origin xyz="0 0 0"/>
-    <geometry>
-      <box size="0.3 0.2 0.1" />
-    </geometry>
-  </visual>
-  <collision>
-    <origin xyz="0 0 0"/>
-    <geometry>
-      <box size="0.3 0.2 0.1" />
-    </geometry>
-  </collision>
+    <inertial>
+      <origin xyz="0 0 0" />
+      <mass value="5" />
+      <inertia  ixx="0.1" ixy="0.0"  ixz="0.0"  iyy="0.1"  iyz="0.0"  izz="0.1" />
+    </inertial>
+    <visual>
+      <origin xyz="0 0 0"/>
+      <geometry>
+        <box size="0.3 0.2 0.1" />
+      </geometry>
+    </visual>
+    <collision>
+      <origin xyz="0 0 0"/>
+      <geometry>
+        <box size="0.3 0.2 0.1" />
+      </geometry>
+    </collision>
   </link>
   <joint name="base_link_box" type="fixed">
@@ -56,21 +56,21 @@
   </gazebo>
   <link name="right_wheel">
-  <inertial>
-    <origin rpy="1.5707963267948966 0 0" xyz="0 0 0" />
-    <mass value="0.1" />
-    <inertia  ixx="0.01" ixy="0.0"  ixz="0.0"  iyy="0.01"  iyz="0.0"  izz="0.01" />
-  </inertial>
-  <visual>
-    <origin rpy="1.5707963267948966 0 0" xyz="0 0 0"/>
-    <geometry>
-      <cylinder length="0.05" radius="0.075"/>
-    </geometry>
-  </visual>
-  <collision>
-    <origin rpy="1.5707963267948966 0 0" xyz="0 0 0"/>
-    <geometry>
-      <cylinder length="0.05" radius="0.075"/>
-    </geometry>
-  </collision>
+    <inertial>
+      <origin rpy="1.5707963267948966 0 0" xyz="0 0 0" />
+      <mass value="0.1" />
+      <inertia  ixx="0.01" ixy="0.0"  ixz="0.0"  iyy="0.01"  iyz="0.0"  izz="0.01" />
+    </inertial>
+    <visual>
+      <origin rpy="1.5707963267948966 0 0" xyz="0 0 0"/>
+      <geometry>
+        <cylinder length="0.05" radius="0.075"/>
+      </geometry>
+    </visual>
+    <collision>
+      <origin rpy="1.5707963267948966 0 0" xyz="0 0 0"/>
+      <geometry>
+        <cylinder length="0.05" radius="0.075"/>
+      </geometry>
+    </collision>
   </link>
   <gazebo reference="right_wheel">
@@ -94,21 +94,21 @@
   </transmission>
   <link name="left_wheel">
-  <inertial>
-    <origin rpy="1.5707963267948966 0 0" xyz="0 0 0" />
-    <mass value="0.1" />
-    <inertia  ixx="0.01" ixy="0.0"  ixz="0.0"  iyy="0.01"  iyz="0.0"  izz="0.01" />
-  </inertial>
-  <visual>
-    <origin rpy="1.5707963267948966 0 0" xyz="0 0 0"/>
-    <geometry>
-      <cylinder length="0.05" radius="0.075"/>
-    </geometry>
-  </visual>
-  <collision>
-    <origin rpy="1.5707963267948966 0 0" xyz="0 0 0"/>
-    <geometry>
-      <cylinder length="0.05" radius="0.075"/>
-    </geometry>
-  </collision>
+    <inertial>
+      <origin rpy="1.5707963267948966 0 0" xyz="0 0 0" />
+      <mass value="0.1" />
+      <inertia  ixx="0.01" ixy="0.0"  ixz="0.0"  iyy="0.01"  iyz="0.0"  izz="0.01" />
+    </inertial>
+    <visual>
+      <origin rpy="1.5707963267948966 0 0" xyz="0 0 0"/>
+      <geometry>
+        <cylinder length="0.05" radius="0.075"/>
+      </geometry>
+    </visual>
+    <collision>
+      <origin rpy="1.5707963267948966 0 0" xyz="0 0 0"/>
+      <geometry>
+        <cylinder length="0.05" radius="0.075"/>
+      </geometry>
+    </collision>
   </link>
   <gazebo reference="left_wheel">
@@ -132,21 +132,21 @@
   </transmission>
   <link name="back_wheel">
-  <inertial>
-    <origin rpy="1.5707963267948966 0 0" xyz="0 0 0" />
-    <mass value="0.1" />
-    <inertia  ixx="0.01" ixy="0.0"  ixz="0.0"  iyy="0.01"  iyz="0.0"  izz="0.01" />
-  </inertial>
-  <visual>
-    <origin rpy="1.5707963267948966 0 0" xyz="0 0 0"/>
-    <geometry>
-      <sphere length="0.1" radius="0.03"/>
-    </geometry>
-  </visual>
-  <collision>
-    <origin rpy="1.5707963267948966 0 0" xyz="0 0 0"/>
-    <geometry>
-      <sphere length="0.1" radius="0.03"/>
-    </geometry>
-  </collision>
+    <inertial>
+      <origin rpy="1.5707963267948966 0 0" xyz="0 0 0" />
+      <mass value="0.1" />
+      <inertia  ixx="0.01" ixy="0.0"  ixz="0.0"  iyy="0.01"  iyz="0.0"  izz="0.01" />
+    </inertial>
+    <visual>
+      <origin rpy="1.5707963267948966 0 0" xyz="0 0 0"/>
+      <geometry>
+        <sphere length="0.1" radius="0.03"/>
+      </geometry>
+    </visual>
+    <collision>
+      <origin rpy="1.5707963267948966 0 0" xyz="0 0 0"/>
+      <geometry>
+        <sphere length="0.1" radius="0.03"/>
+      </geometry>
+    </collision>
       <surface>
         <friction>
@@ -251,4 +251,5 @@
     <wheelSeparation>0.35</wheelSeparation>
     <wheelDiameter>0.15</wheelDiameter>
+    <legacyMode> true </legacyMode>
     <torque>1.41</torque>
     <commandTopic>cmd_vel</commandTopic>

File: urdf/hokuyo.xacro (robot description, xacro)
@@ -1,4 +1,5 @@
 <?xml version="1.0"?>
 <robot xmlns:xacro="http://www.ros.org/wiki/xacro">
+<xacro:property name="M_PI" value="3.1415926535897931" />
 <!-- Front Laser -->
 <xacro:macro name="laser" params="name parent xyz rpy meshes" >
@@ -61,3 +62,66 @@
     </gazebo>
 </xacro:macro>
+<!-- Front camera -->
+<xacro:macro name="camera_link" params="parent">
+  <link name="camera_link">
+    <collision>
+      <origin xyz="0 0 0" rpy="0 0 0" />
+      <geometry>
+        <mesh filename="package://sensors_and_actuators/meshes/camara.stl" scale="0.1 0.1 0.1"/>
+      </geometry>
+    </collision>
+    <visual>
+      <origin xyz="0 0 0" rpy="0 0 0" />
+      <geometry>
+        <mesh filename="package://sensors_and_actuators/meshes/camara.stl" scale="0.1 0.1 0.1"/>
+      </geometry>
+      <material name="grey">
+          <color rgba="0.2 0.2 0.2 1.0"/>
+      </material>
+    </visual>
+    <inertial>
+      <mass value="0.001" />
+      <origin xyz="0 0 0" rpy="0 0 0" />
+      <inertia ixx="0.0001" ixy="0" ixz="0" iyy="0.0001" iyz="0" izz="0.0001" />
+    </inertial>
+  </link>
+  <joint name="camera_joint" type="fixed">
+      <parent link="${parent}"/>
+      <child link="camera_link"/>
+      <origin rpy="0 0 0" xyz="0.047 0.0 0.0"/>
+      <axis xyz="1 0 0" />
+  </joint>
+  <gazebo reference="camera_link">
+    <sensor type="camera" name="camera_camera_sensor">
+      <update_rate>30.0</update_rate>
+      <camera>
+        <pose>0.035 0 0.078 0 ${-M_PI/2} 0</pose>
+        <horizontal_fov>${85 * M_PI/180.0}</horizontal_fov>
+        <image>
+          <format>R8G8B8</format>
+          <width>1020</width>
+          <height>1020</height>
+        </image>
+        <clip>
+          <near>0.01</near>
+          <far>100</far>
+        </clip>
+      </camera>
+      <plugin name="camera_camera_controller" filename="libgazebo_ros_camera.so">
+        <alwaysOn>true</alwaysOn>
+        <updateRate>0.0</updateRate>
+        <cameraName>arm_sensor/camera</cameraName>
+        <imageTopicName>image_raw</imageTopicName>
+        <cameraInfoTopicName>camera_info</cameraInfoTopicName>
+        <frameName>camera_link</frameName>
+        <hackBaseline>0.07</hackBaseline>
+        <distortionK1>0.0</distortionK1>
+        <distortionK2>0.0</distortionK2>
+        <distortionK3>0.0</distortionK3>
+        <distortionT1>0.0</distortionT1>
+        <distortionT2>0.0</distortionT2>
+      </plugin>
+    </sensor>
+  </gazebo>
+</xacro:macro>
 </robot>

Commit message: Added camera and configured it, need to write a node to use the camera raw data. going to sleep :P
Signed-off-by: lidorshimoni <lidor.shim@gmail.com>

File: urdf/ABot.urdf.xacro (robot description, xacro)
@@ -27,4 +27,30 @@
     </collision>
   </link>
+    <link name="camera_link">
+    <collision>
+      <origin xyz="0 0 0" rpy="0 0 0"/>
+      <geometry>
+    <box size="0.01 0.01 0.01"/>
+      </geometry>
+    </collision>
+    <visual>
+      <origin xyz="0 0 0" rpy="0 0 0"/>
+      <geometry>
+    <box size="0.01 0.01 0.01"/>
+      </geometry>
+      <material name="red"/>
+    </visual>
+    <inertial>
+      <mass value="1e-5" />
+      <origin xyz="0 0 0" rpy="0 0 0"/>
+      <inertia ixx="1e-6" ixy="0" ixz="0" iyy="1e-6" iyz="0" izz="1e-6" />
+    </inertial>
+  </link>
+  <joint name="camera_joint" type="fixed">
+    <axis xyz="0 1 0" />
+    <origin xyz="0.23 0 0.25" rpy="0 0 0"/>
+    <parent link="base_link"/>
+    <child link="camera_link"/>
+  </joint>
   <link name="box">
     <inertial>
@@ -243,4 +269,44 @@
     </joint>
   </transmission-->
+<!-- camera -->
+  <gazebo reference="camera_link">
+    <sensor type="camera" name="camera1">
+      <update_rate>30.0</update_rate>
+      <camera name="head">
+        <horizontal_fov>1.3962634</horizontal_fov>
+        <image>
+          <width>800</width>
+          <height>800</height>
+          <format>R8G8B8</format>
+        </image>
+        <clip>
+          <near>0.02</near>
+          <far>300</far>
+        </clip>
+        <noise>
+          <type>gaussian</type>
+          <!-- Noise is sampled independently per pixel on each frame.
+               That pixel's noise value is added to each of its color
+               channels, which at that point lie in the range [0,1]. -->
+          <mean>0.0</mean>
+          <stddev>0.007</stddev>
+        </noise>
+      </camera>
+      <plugin name="camera_controller" filename="libgazebo_ros_camera.so">
+        <alwaysOn>true</alwaysOn>
+        <updateRate>0.0</updateRate>
+        <cameraName>/camera</cameraName>
+        <imageTopicName>image_raw</imageTopicName>
+        <cameraInfoTopicName>camera_info</cameraInfoTopicName>
+        <frameName>camera_link</frameName>
+        <hackBaseline>0.07</hackBaseline>
+        <distortionK1>0.0</distortionK1>
+        <distortionK2>0.0</distortionK2>
+        <distortionK3>0.0</distortionK3>
+        <distortionT1>0.0</distortionT1>
+        <distortionT2>0.0</distortionT2>
+      </plugin>
+    </sensor>
+  </gazebo>
 <gazebo>
   <plugin name="differential_drive_controller" filename="libgazebo_ros_diff_drive.so">
@@ -261,5 +327,6 @@
   </plugin>
 </gazebo>
-  <xacro:include filename="$(find SLAM)/urdf/hokuyo.xacro"/>
+  <xacro:include filename="$(find Fire_Fighting_Robot)/urdf/hokuyo.xacro"/>
   <xacro:laser name="base_laser" parent="base_link" xyz="0.225 0 0.2" rpy="0 0 0" meshes="package://gazebo_plugins/test/multi_robot_scenario/meshes/laser"/>
+  <xacro:property name="camera_link" value="0.05" /> <!-- Size of square 'camera' box -->
 </robot>

File: urdf/camera.xacro (robot description, xacro)
@@ -1,7 +1,6 @@
 <?xml version="1.0"?>
 <robot xmlns:xacro="http://www.ros.org/wiki/xacro">
-<xacro:property name="M_PI" value="3.1415926535897931" />
-<!-- Front Laser -->
-<xacro:macro name="laser" params="name parent xyz rpy meshes" >
+<!-- Front Camera -->
+<xacro:macro name="camera" params="name parent xyz rpy meshes" >
   <joint name="${parent}_${name}_joint" type="fixed">
       <axis xyz="0 0 1" />

Commit message: Changed the robot to KoBot for better stability, some bugs still need fixing.
Signed-off-by: lidorshimoni <lidor.shim@gmail.com>

File: urdf/ABot.urdf.xacro (robot description, xacro)
@@ -27,5 +27,5 @@
     </collision>
   </link>
-    <link name="camera_link">
+  <link name="camera_link">
     <collision>
       <origin xyz="0 0 0" rpy="0 0 0"/>

File: urdf/KoBot.urdf.xacro (robot description, xacro)
@@ -54,21 +54,21 @@
   </joint>
   <link name="box">
-  <inertial>
-    <origin xyz="0 0 0" />
-    <mass value="5" />
-    <inertia  ixx="0.1" ixy="0.0"  ixz="0.0"  iyy="0.1"  iyz="0.0"  izz="0.1" />
-  </inertial>
-  <visual>
-    <origin xyz="0 0 0"/>
-    <geometry>
-      <box size="0.3 0.2 0.1" />
-    </geometry>
-  </visual>
-  <collision>
-    <origin xyz="0 0 0"/>
-    <geometry>
-      <box size="0.3 0.2 0.1" />
-    </geometry>
-  </collision>
+    <inertial>
+      <origin xyz="0 0 0" />
+      <mass value="5" />
+      <inertia  ixx="0.1" ixy="0.0"  ixz="0.0"  iyy="0.1"  iyz="0.0"  izz="0.1" />
+    </inertial>
+    <visual>
+      <origin xyz="0 0 0"/>
+      <geometry>
+        <box size="0.3 0.2 0.1" />
+      </geometry>
+    </visual>
+    <collision>
+      <origin xyz="0 0 0"/>
+      <geometry>
+        <box size="0.3 0.2 0.1" />
+      </geometry>
+    </collision>
   </link>
   <joint name="base_link_box" type="fixed">
@@ -82,21 +82,21 @@
   </gazebo>
   <link name="right_wheel">
-  <inertial>
-    <origin rpy="1.5707963267948966 0 0" xyz="0 0 0" />
-    <mass value="0.1" />
-    <inertia  ixx="0.01" ixy="0.0"  ixz="0.0"  iyy="0.01"  iyz="0.0"  izz="0.01" />
-  </inertial>
-  <visual>
-    <origin rpy="1.5707963267948966 0 0" xyz="0 0 0"/>
-    <geometry>
-      <cylinder length="0.05" radius="0.075"/>
-    </geometry>
-  </visual>
-  <collision>
-    <origin rpy="1.5707963267948966 0 0" xyz="0 0 0"/>
-    <geometry>
-      <cylinder length="0.05" radius="0.075"/>
-    </geometry>
-  </collision>
+    <inertial>
+      <origin rpy="1.5707963267948966 0 0" xyz="0 0 0" />
+      <mass value="0.1" />
+      <inertia  ixx="0.01" ixy="0.0"  ixz="0.0"  iyy="0.01"  iyz="0.0"  izz="0.01" />
+    </inertial>
+    <visual>
+      <origin rpy="1.5707963267948966 0 0" xyz="0 0 0"/>
+      <geometry>
+        <cylinder length="0.05" radius="0.075"/>
+      </geometry>
+    </visual>
+    <collision>
+      <origin rpy="1.5707963267948966 0 0" xyz="0 0 0"/>
+      <geometry>
+        <cylinder length="0.05" radius="0.075"/>
+      </geometry>
+    </collision>
   </link>
   <gazebo reference="right_wheel">
@@ -120,21 +120,21 @@
   </transmission>
   <link name="left_wheel">
-  <inertial>
-    <origin rpy="1.5707963267948966 0 0" xyz="0 0 0" />
-    <mass value="0.1" />
-    <inertia  ixx="0.01" ixy="0.0"  ixz="0.0"  iyy="0.01"  iyz="0.0"  izz="0.01" />
-  </inertial>
-  <visual>
-    <origin rpy="1.5707963267948966 0 0" xyz="0 0 0"/>
-    <geometry>
-      <cylinder length="0.05" radius="0.075"/>
-    </geometry>
-  </visual>
-  <collision>
-    <origin rpy="1.5707963267948966 0 0" xyz="0 0 0"/>
-    <geometry>
-      <cylinder length="0.05" radius="0.075"/>
-    </geometry>
-  </collision>
+    <inertial>
+      <origin rpy="1.5707963267948966 0 0" xyz="0 0 0" />
+      <mass value="0.1" />
+      <inertia  ixx="0.01" ixy="0.0"  ixz="0.0"  iyy="0.01"  iyz="0.0"  izz="0.01" />
+    </inertial>
+    <visual>
+      <origin rpy="1.5707963267948966 0 0" xyz="0 0 0"/>
+      <geometry>
+        <cylinder length="0.05" radius="0.075"/>
+      </geometry>
+    </visual>
+    <collision>
+      <origin rpy="1.5707963267948966 0 0" xyz="0 0 0"/>
+      <geometry>
+        <cylinder length="0.05" radius="0.075"/>
+      </geometry>
+    </collision>
   </link>
   <gazebo reference="left_wheel">
@@ -321,5 +321,5 @@
     <odometryTopic>odom</odometryTopic>
     <odometryFrame>odom</odometryFrame>
-    <robotBaseFrame>base_link</robotBaseFrame>
+    <robotBaseFrame>base_linsk</robotBaseFrame>
     <publishWheelJointState>true</publishWheelJointState>
   </plugin>
@@ -338,3 +338,4 @@
   <xacro:include filename="$(find fire_fighting_robot)/urdf/hokuyo.xacro"/>
   <xacro:laser name="base_laser" parent="base_link" xyz="0.225 0 0.2" rpy="0 0 0" meshes="package://gazebo_plugins/test/multi_robot_scenario/meshes/laser"/>
+  <!-- <xacro:property name="camera_link" value="0.05" /> Size of square 'camera' box -->
 </robot>
